File: hardware/nrf52-co2-sensor/nrf52-co2-sensor.kicad_sch (KiCad schematic)
At the start: 33 parts, among them J1 USB4105-GF-A, J2 SCD30, J3 Conn_01x03, J4 SWD, J5 Filter_Bypass, Q2 Q_NPN_BEC, SW1 SW_Push, U1 USBLC6-2P6, U2 MDBT50Q-1MV2

Commit message: Finished PCB Layout and BOM read for review
Parts:
- removed J5: Filter_Bypass, symbol Connector:Conn_01x02_Pin
- added J6: Conn_01x02, Connector_JST:JST_XH_B2B-XH-AM_1x02_P2.50mm_Vertical, symbol Connector_Generic:Conn_01x02
- added J7: Conn_01x02, Connector_PinHeader_2.54mm:PinHeader_1x02_P2.54mm_Vertical, symbol Connector_Generic:Conn_01x02
- C10: Digikey (none) -> https://www.digikey.com/en/products/detail/murata-electroni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; Digikey_PartNumber (none) -> 490-1313-1-ND
- C3: Digikey https://www.digikey.com/en/products/detail/nextgen-componen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 -> https://www.digikey.com/en/products/detail/murata-electroni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; Digikey_PartNumber (none) -> 490-GRM155R61A225KE01JCT-ND
- C4, C9: Digikey (none) -> https://www.digikey.com/en/products/detail/murata-electroni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; Digikey_PartNumber (none) -> 490-3261-1-ND
- C5: value 100nF -> 0.1uf; Digikey (none) -> https://www.digikey.com/en/products/detail/murata-electroni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; Digikey_PartNumber (none) -> 490-3261-1-ND
- C6: footprint Capacitor_SMD:C_0402_1005Metric -> Capacitor_SMD:C_0805_2012Metric; Digikey (none) -> https://www.digikey.com/en/products/detail/samsung-electro-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; Digikey_PartNumber (none) -> 1276-1052-1-ND; KiLib_Generator (none) -> SMD_2terminal_chip_molded
- C7: footprint Capacitor_SMD:C_0402_1005Metric -> Capacitor_SMD:C_0805_2012Metric; Digikey (none) -> https://www.digikey.com/en/products/detail/samsung-electro-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; Digikey_PartNumber (none) -> 1276-1052-1-ND
- C8: footprint Capacitor_SMD:C_0402_1005Metric -> Capacitor_SMD:C_1206_3216Metric; Digikey https://www.digikey.com/en/products/detail/nextgen-componen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 -> https://www.digikey.com/en/products/detail/murata-electroni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; Digikey_PartNumber (none) -> 490-9673-1-ND; KiLib_Generator (none) -> SMD_2terminal_chip_molded
- D1, D2: Digikey_PartNumber (none) -> 160-LTST-C190GKTCT-ND
- D3: footprint Diode_THT:D_DO-35_SOD27_P7.62mm_Horizontal -> Diode_SMD:D_SOD-123; Digikey (none) -> https://www.digikey.com/en/products/detail/mcc-micro-commer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; Digikey_PartNumber (none) -> 1N4148WTPMSCT-ND
- J1: Digikey (none) -> https://www.digikey.com/en/products/detail/gct/USB4105-GF-A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; Digikey_PartNumber (none) -> 2073-USB4105-GF-ACT-ND; digikey https://www.digikey.com/en/products/detail/gct/USB4105-GF-A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 -> (none)
- J2: footprint Connector_PinHeader_1.00mm:PinHeader_1x05_P1.00mm_Vertical -> Connector_PinHeader_2.54mm:PinHeader_1x05_P2.54mm_Vertical; Digikey (none) -> https://www.digikey.com/en/products/detail/sullins-connecto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; Digikey_PartNumber (none) -> S1012E-05-ND
- J3: footprint (none) -> Connector_PinHeader_2.54mm:PinHeader_1x03_P2.54mm_Vertical; Digikey (none) -> https://www.digikey.com/en/products/detail/sullins-connecto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; Digikey_PartNumber (none) -> S1012E-03-ND; KiLib_Generator (none) -> connector/pin_header_socket
- J4: footprint Connector_PinHeader_1.00mm:PinHeader_1x05_P1.00mm_Vertical -> Connector_PinHeader_2.54mm:PinHeader_1x05_P2.54mm_Vertical; Digikey https://www.digikey.com/en/products/detail/digikey-va/316-4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 -> https://www.digikey.com/en/products/detail/sullins-connecto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; Digikey_PartNumber (none) -> S1012E-05-ND
- L1: footprint Inductor_SMD:L_0402_1005Metric -> Inductor_SMD:L_0805_2012Metric; Digikey (none) -> https://www.digikey.com/en/products/detail/tdk/MLZ2012N100L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; Digikey_PartNumber (none) -> 445-6762-1-ND
- Q2: value Q_NPN_BEC -> MMBT2222A-TP; footprint (none) -> Package_TO_SOT_SMD:SOT-23; Digikey (none) -> https://www.digikey.com/en/products/detail/mcc-micro-commer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; Digikey_PartNumber (none) -> MMBT2222ATPMSCT-ND; KiLib_Generator (none) -> package/gullwing
- R1, R2: Digikey (none) -> https://www.digikey.com/en/products/detail/yageo/RC0402FR-0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; Digikey_PartNumber (none) -> 311-5.10KLRCT-ND; digikey https://www.digikey.com/en/products/detail/yageo/RC0603FR-0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 -> (none)
- R10: Digikey (none) -> https://www.digikey.com/en/products/detail/yageo/RC0402FR-0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; Digikey_PartNumber (none) -> 311-150LRCT-ND
- R11: Digikey (none) -> https://www.digikey.com/en/products/detail/yageo/RC0402FR-0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; Digikey_PartNumber (none) -> 13-RC0402FR-072M2LCT-ND; digikey https://www.digikey.com/en/products/detail/yageo/RC0603FR-0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 -> (none)
- R12: Digikey (none) -> https://www.digikey.com/en/products/detail/yageo/RC0402FR-0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; Digikey_PartNumber (none) -> 311-1.00MLRCT-ND; digikey https://www.digikey.com/en/products/detail/yageo/RC0603FR-0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 -> (none)
- R3, R4: Digikey (none) -> https://www.digikey.com/en/products/detail/yageo/RC0402FR-0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; Digikey_PartNumber (none) -> 311-22.0LRCT-ND
- R5, R6, R9: Digikey (none) -> https://www.digikey.com/en/products/detail/yageo/RC0402FR-0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; Digikey_PartNumber (none) -> 311-4.7KLRCT-ND
- R7: Digikey (none) -> https://www.digikey.com/en/products/detail/yageo/RC0402FR-0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; Digikey_PartNumber (none) -> 311-10.0KLRCT-ND
- R8: Digikey (none) -> https://www.digikey.com/en/products/detail/yageo/RC0402FR-0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; Digikey_PartNumber (none) -> 311-2.20KLRCT-ND
- SW1: footprint SW4_SKRPABE010_ALPS -> nrf52-co2-sensor:SW4_SKRPABE010_ALPS; Digikey https://www.digikey.com/en/products/detail/alps-alpine/SKRP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 -> https://www.digikey.com/en/products/detail/same-sky-formerl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; Digikey_PartNumber (none) -> 2223-TS20-42-25-WT-160-SMT-TRCT-ND
- U1: Digikey (none) -> https://www.digikey.com/en/products/detail/stmicroelectroni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; Digikey_PartNumber (none) -> 497-5026-1-ND; digikey https://www.digikey.com/en/products/detail/stmicroelectroni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 -> (none)
- U2: Digikey_PartNumber (none) -> 3271-MDBT50Q-1MV2-ND
Connections:
- net External Power: now also J6.1 (Pin_1)
- net GND: now also C7.2, J6.2 (Pin_2); no longer C7.1
- net POWER_RAW: now also J7.2 (Pin_2)
- net POWER_SENS: now also J7.1 (Pin_1)
- net VBUS: now also C7.1; no longer C7.2
- net CC2: now reaches J1.B5 (CC2), R2.1
- net BASE: now reaches C8.2, D3.1 (K), Q2.1 (B), R10.1
- net D1+: now reaches R3.2, U1.4 (I/O2)
- net D1-: now reaches R4.1, U1.6 (I/O1)
- net CC1: now reaches J1.A5 (CC1), R1.1
- net D+_MCU renamed D_MCU+
- net D-_MCU renamed D_MCU-
